File: PiVideoCapturer.sch (KiCad schematic (older format))
At the start: 41 parts, among them J1 HDMI, J2 Conn_01x09_Female, J3 MIPI_30PIN, J4 MIPI_30PIN, U1 TC358840XBG, U2 AP2127K-ADJTRG1, U3 AP2127K-ADJTRG1, U4 AP2127K-ADJTRG1, X1 SG-310SCF

Commit message: BOM: add FPC 30P 0.5mm vertical
Parts:
- J3, J4: SuppliersPartNumber N/A -> C11078
Changed lines of the file:
@@
 F 2 "pi_video_capturer:MIPI_30PIN_FPC_0.5mm" H 10141 2401 50  0001 L BNN
 F 3 "" H 10141 2401 50  0001 L BNN
-F 4 "N/A" V 10141 2401 50  0001 C CNN "SuppliersPartNumber"
+F 4 " C11078" V 10141 2401 50  0001 C CNN "SuppliersPartNumber"
 	1    10141 2401
 	0    1    1    0
@@
 F 2 "pi_video_capturer:MIPI_30PIN_FPC_0.5mm" H 8561 2396 50  0001 L BNN
 F 3 "" H 8561 2396 50  0001 L BNN
-F 4 "N/A" V 8561 2396 50  0001 C CNN "SuppliersPartNumber"
+F 4 " C11078" V 8561 2396 50  0001 C CNN "SuppliersPartNumber"
 	1    8561 2396
 	0    1    1    0

Commit message: bom: add TC358840XBG part number
Parts:
- U1: SuppliersPartNumber (none) -> C2764727
Changed lines of the file:
@@
 F 2 "pi_video_capturer:BGA80C65P10X10_700X700X100N" H 5466 2770 50  0001 C CNN
 F 3 "" H 5466 2770 50  0001 C CNN
+F 4 "C2764727" H 5366 2720 50  0001 C CNN "SuppliersPartNumber"
 	1    5366 2720
 	1    0    0    -1
